File: kicad/STM32_IEEE488_USB/STM32_IEEE488_USB.kicad_sch (KiCad schematic)
At the start: 14 parts, among them J1 Conn_02x23_Odd_Even, J4 HEADER, J5 IEEE488, J7 STM32F401, U1 SN75162BN, U4 SN75160BN

Commit message: pinout fixed
Connections:
- net PE#: now also J7.13 (Pin_13); no longer J7.22 (Pin_22)
- new net LED: J7.22 (Pin_22)
Changed lines of the file:
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@@
 	)
 	(label "PE#"
-		(at 63.5 176.53 180)
+		(at 31.75 161.29 0)
 		(effects
 			(font
 				(size 1.27 1.27)
 			)
-			(justify right bottom)
+			(justify left bottom)
 		)
 	)
@@
 		(effects
 			(font
+				(size 1.27 1.27)
+			)
+			(justify right bottom)
+		)
+	)
+	(label "LED"
+		(at 63.5 176.53 180)
+		(effects
+			(font

Commit message: final pin arrangement
Connections:
- net DET_SD is gone; now on net NDAC#: J7.5 (Pin_5)
- net MISO_SD is gone; now on net PE#: J7.3 (Pin_3)
- net MOSI_SD is gone; now on net IFC#: J7.4 (Pin_4)
- net SCK_SD is gone; now on net DAV#: J7.2 (Pin_2)
- net ~{CS_SD} is gone; now on net EOI#: J7.1 (Pin_1)
- net DAV#: no longer J7.12 (Pin_12)
- net DIO1#: now also J7.34 (Pin_34); no longer J7.26 (Pin_26)
- net DIO2#: now also J7.35 (Pin_35); no longer J7.27 (Pin_27)
- net DIO3#: now also J7.36 (Pin_36); no longer J7.28 (Pin_28)
- net DIO4#: now also J7.11 (Pin_11); no longer J7.29 (Pin_29)
- net DIO5#: now also J7.12 (Pin_12); no longer J7.30 (Pin_30)
- net DIO6#: now also J7.13 (Pin_13); no longer J7.31 (Pin_31)
- net DIO7#: now also J7.14 (Pin_14); no longer J7.32 (Pin_32)
- net DIO8#: now also J7.15 (Pin_15); no longer J7.33 (Pin_33)
- net EOI#: no longer J7.11 (Pin_11)
- net IFC#: no longer J7.35 (Pin_35)
- net NDAC#: no longer J7.36 (Pin_36)
- net PE#: no longer J7.13 (Pin_13)
- net REN#: now also J7.27 (Pin_27); no longer J7.34 (Pin_34)
- net SCL: now reaches J7.16 (Pin_16)
- net SDA: now reaches J7.17 (Pin_17)
- new net BUTTON: J7.26 (Pin_26)
- new net DEBUG1: J7.30 (Pin_30)
- new net MISO: J7.32 (Pin_32)
- new net MOSI: J7.33 (Pin_33)
- new net RX2: J7.29 (Pin_29)
- new net SCK: J7.31 (Pin_31)
- new net TX2: J7.28 (Pin_28)
- no-connect marks 10 -> 18
Other:
- note added: "B12 B13 B14 B15 A8 A9 A10 USB A11 USB A12 A15 B3 B4 B5 B6 B7 B8 B9"
- note removed: "B12 B13 B14 B15 A8 A9 A10 USB A11 USB A12 A15 B3 B4 B5 SCL B6 SDA B7 B8 B9"
- note removed: "SDCARD"
Changed lines of the file:
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@@
 		)
 	)
-	(text "B12\nB13\nB14\nB15\nA8\nA9\nA10\nUSB A11\nUSB A12\nA15\nB3\nB4\nB5\nSCL B6\nSDA B7\nB8\nB9"
+	(text "B12\nB13\nB14\nB15\nA8\nA9\nA10\nUSB A11\nUSB A12\nA15\nB3\nB4\nB5\nB6\nB7\nB8\nB9"
 		(exclude_from_sim no)
-		(at 19.304 170.688 0)
+		(at 21.082 171.196 0)
 		(effects
 			(font
-				(size 1.55 1.55)
+				(size 1.5748 1.5748)
 			)
 			(justify left bottom)
 		)
 	)
-	(text "SDCARD"
-		(exclude_from_sim no)
-		(at 26.162 134.112 90)
-		(effects
-			(font
-				(size 1.27 1.27)
-			)
-		)
-	)
 	(text "STM32F401\nmicrocontroller"
 		(exclude_from_sim no)
@@
 	)
 	(no_connect
+		(at 31.75 171.45)
+	)
+	(no_connect
+		(at 63.5 148.59)
+	)
+	(no_connect
 		(at 228.6 135.89)
 	)
@@
 	)
 	(no_connect
+		(at 63.5 158.75)
+	)
+	(no_connect
 		(at 41.91 148.59)
 	)
 	(no_connect
+		(at 31.75 168.91)
+	)
+	(no_connect
+		(at 63.5 153.67)
+	)
+	(no_connect
 		(at 54.61 135.89)
 	)
@@
 	)
 	(no_connect
+		(at 63.5 166.37)
+	)
+	(no_connect
 		(at 54.61 133.35)
 	)
@@
 	)
 	(no_connect
+		(at 63.5 151.13)
+	)
+	(no_connect
+		(at 63.5 161.29)
+	)
+	(no_connect
 		(at 54.61 130.81)
 	)
@@
 	(wire
 		(pts
-			(xy 29.21 130.81) (xy 41.91 130.81)
+			(xy 31.75 130.81) (xy 41.91 130.81)
 		)
 		(stroke
@@
 	(wire
 		(pts
-			(xy 29.21 135.89) (xy 41.91 135.89)
+			(xy 31.75 135.89) (xy 41.91 135.89)
 		)
 		(stroke
@@
 	(wire
 		(pts
-			(xy 29.21 140.97) (xy 41.91 140.97)
+			(xy 31.75 140.97) (xy 41.91 140.97)
 		)
 		(stroke
@@
 	(wire
 		(pts
-			(xy 29.21 133.35) (xy 41.91 133.35)
+			(xy 31.75 133.35) (xy 41.91 133.35)
 		)
 		(stroke
@@
 	(wire
 		(pts
-			(xy 29.21 138.43) (xy 41.91 138.43)
+			(xy 31.75 138.43) (xy 41.91 138.43)
 		)
 		(stroke
@@
 		)
 	)
-	(polyline
-		(pts
-			(xy 27.94 128.27) (xy 27.94 140.97)
-		)
-		(stroke
-			(width 0)
-			(type default)
-		)
-	)
 	(wire
 		(pts
@@
 		)
 	)
-	(label "MOSI_SD"
-		(at 29.21 138.43 0)
+	(label "DIO6"
+		(at 247.65 110.49 180)
 		(effects
 			(font
 				(size 1.27 1.27)
 			)
-			(justify left bottom)
+			(justify right bottom)
 		)
 	)
-	(label "DIO6"
-		(at 247.65 110.49 180)
+	(label "~{STMRST}"
+		(at 63.5 168.91 180)
 		(effects
 			(font
@@
 		)
 	)
-	(label "~{STMRST}"
-		(at 63.5 168.91 180)
+	(label "SCL"
+		(at 31.75 168.91 0)
 		(effects
 			(font
 				(size 1.27 1.27)
 			)
-			(justify right bottom)
+			(justify left bottom)
 		)
 	)
@@
 	)
 	(label "DAV#"
-		(at 31.75 158.75 0)
+		(at 31.75 133.35 0)
 		(effects
 			(font
@@
 		)
 	)
+	(label "~{CSFLSH}"
+		(at 80.01 156.21 180)
+		(effects
+			(font
+				(size 1.27 1.27)
+			)
+			(justify right bottom)
+		)
+	)
 	(label "PE#"
-		(at 31.75 161.29 0)
+		(at 31.75 135.89 0)
 		(effects
 			(font
@@
 		)
 	)
-	(label "SCK_SD"
-		(at 29.21 133.35 0)
-		(effects
-			(font
-				(size 1.27 1.27)
-			)
-			(justify left bottom)
-		)
-	)
 	(label "DIO2#"
 		(at 128.27 100.33 180)
@@
 	)
 	(label "DIO4#"
-		(at 63.5 158.75 180)
+		(at 31.75 156.21 0)
 		(effects
 			(font
 				(size 1.27 1.27)
 			)
-			(justify right bottom)
+			(justify left bottom)
 		)
 	)
@@
 	)
 	(label "DIO3#"
-		(at 63.5 161.29 180)
+		(at 63.5 140.97 180)
 		(effects
 			(font
@@
 		)
 	)
-	(label "~{CS_SD}"
-		(at 29.21 130.81 0)
-		(effects
-			(font
-				(size 1.27 1.27)
-			)
-			(justify left bottom)
-		)
-	)
 	(label "DIO8"
 		(at 210.82 135.89 180)
@@
 		)
 	)
+	(label "MISO"
+		(at 63.5 151.13 180)
+		(effects
+			(font
+				(size 1.27 1.27)
+			)
+			(justify right bottom)
+		)
+	)
 	(label "DIO3#"
 		(at 128.27 97.79 180)
@@
 	)
 	(label "DIO7#"
-		(at 63.5 151.13 180)
+		(at 31.75 163.83 0)
 		(effects
 			(font
 				(size 1.27 1.27)
 			)
-			(justify right bottom)
+			(justify left bottom)
 		)
 	)
@@
 	)
 	(label "EOI#"
-		(at 31.75 156.21 0)
+		(at 31.75 130.81 0)
 		(effects
 			(font
@@
 		)
 	)
+	(label "RX2"
+		(at 63.5 158.75 180)
+		(effects
+			(font
+				(size 1.27 1.27)
+			)
+			(justify right bottom)
+		)
+	)
 	(label "DIO1#"
 		(at 128.27 102.87 180)
@@
 	)
 	(label "REN#"
-		(at 63.5 146.05 180)
+		(at 63.5 163.83 180)
+		(effects
+			(font
+				(size 1.27 1.27)
+			)
+			(justify right bottom)
+		)
+	)
+	(label "MOSI"
+		(at 63.5 148.59 180)
 		(effects
 			(font
@@
 	)
 	(label "DIO8#"
-		(at 63.5 148.59 180)
+		(at 31.75 166.37 0)
 		(effects
 			(font
 				(size 1.27 1.27)
 			)
-			(justify right bottom)
+			(justify left bottom)
 		)
 	)
@@
 		)
 	)
+	(label "TX2"
+		(at 63.5 161.29 180)
+		(effects
+			(font
+				(size 1.27 1.27)
+			)
+			(justify right bottom)
+		)
+	)
 	(label "DIO1#"
+		(at 63.5 146.05 180)
+		(effects
+			(font
+				(size 1.27 1.27)
+			)
+			(justify right bottom)
+		)
+	)
+	(label "BUTTON"
 		(at 63.5 166.37 180)
 		(effects
@@
 	)
 	(label "DIO6#"
-		(at 63.5 153.67 180)
+		(at 31.75 161.29 0)
 		(effects
 			(font
 				(size 1.27 1.27)
 			)
-			(justify right bottom)
+			(justify left bottom)
 		)
 	)
@@
 		)
 	)
-	(label "DET_SD"
-		(at 29.21 140.97 0)
+	(label "DIO3"
+		(at 223.52 113.03 0)
 		(effects
 			(font
@@
 		)
 	)
-	(label "DIO3"
-		(at 223.52 113.03 0)
+	(label "DIO5#"
+		(at 31.75 158.75 0)
 		(effects
 			(font
@@
 		)
 	)
-	(label "DIO5#"
-		(at 63.5 156.21 180)
+	(label "SDA"
+		(at 31.75 171.45 0)
 		(effects
 			(font
 				(size 1.27 1.27)
 			)
-			(justify right bottom)
+			(justify left bottom)
 		)
 	)
@@
 		)
 	)
-	(label "MISO_SD"
-		(at 29.21 135.89 0)
+	(label "SCK"
+		(at 63.5 153.67 180)
 		(effects
 			(font
 				(size 1.27 1.27)
 			)
-			(justify left bottom)
+			(justify right bottom)
 		)
 	)
@@
 	)
 	(label "IFC#"
-		(at 63.5 143.51 180)
+		(at 31.75 138.43 0)
 		(effects
 			(font
 				(size 1.27 1.27)
 			)
-			(justify right bottom)
+			(justify left bottom)
 		)
 	)
 	(label "DIO2#"
-		(at 63.5 163.83 180)
+		(at 63.5 143.51 180)
 		(effects
 			(font
@@
 		)
 	)
+	(label "DEBUG1"
+		(at 63.5 156.21 180)
+		(effects
+			(font
+				(size 1.27 1.27)
+			)
+			(justify right bottom)
+		)
+	)
 	(label "SRQ#"
 		(at 31.75 146.05 0)
@@
 	)
 	(label "NDAC#"
-		(at 63.5 140.97 180)
+		(at 31.75 140.97 0)
 		(effects
 			(font
 				(size 1.27 1.27)
 			)
-			(justify right bottom)
+			(justify left bottom)
 		)
 	)
